Commit message: make controller

File: src/lookchoop_description/urdf/gazebo_full.xacro (robot description, xacro)
@@ -7,6 +7,6 @@
     <joint name="joint_1">
       <command_interface name="effort">
-        <param name="min">-100</param>
-        <param name="max">100</param>
+        <param name="min">-1000</param>
+        <param name="max">1000</param>
       </command_interface>
       <state_interface name="position">
@@ -18,6 +18,6 @@
     <joint name="joint_2">
       <command_interface name="effort">
-        <param name="min">-100</param>
-        <param name="max">100</param>
+        <param name="min">-1000</param>
+        <param name="max">1000</param>
       </command_interface>
       <state_interface name="position">
@@ -29,6 +29,6 @@
     <joint name="joint_3">
       <command_interface name="effort">
-        <param name="min">-100</param>
-        <param name="max">100</param>
+        <param name="min">-1000</param>
+        <param name="max">1000</param>
       </command_interface>
       <state_interface name="position">

File: src/lookchoop_description/urdf/robot_core.xacro (robot description, xacro)
@@ -7,10 +7,10 @@
     <!-- BASE LINK -->
     <link name="world"/>
-    <!-- <joint name="world_to_base" type="fixed">
+    <joint name="world_to_base" type="fixed">
         <parent link="world"/>
         <child link="base_link"/>
         <origin xyz="0 0 2" rpy="0 0 0"/>
-    </joint> -->
-    <joint name="world_to_base" type="prismatic">
+    </joint>
+    <!-- <joint name="world_to_base" type="prismatic">
         <parent link="world"/>
         <child link="base_link"/>
@@ -18,5 +18,5 @@
         <axis xyz="0 0 1"/>
         <limit effort="1000" velocity="10" lower="-2" upper="2"/>
-    </joint>
+    </joint> -->
     <link name="base_link">
         <visual>
@@ -42,5 +42,5 @@
         <origin xyz="0 0 -${(L_tt/2)+L_td}" rpy="0 0 0"/>
         <axis xyz="0 1 0"/>
-        <limit effort="500" velocity="100" lower="${-PI}" upper="${PI}"/>
+        <limit effort="5000" velocity="100" lower="${-PI}" upper="${PI}"/>
         <dynamics damping="${joint_damping}" friction="${joint_friction}"/>
     </joint>
@@ -68,5 +68,5 @@
         <origin xyz="0 0 -${(L_th)}"/>
         <axis xyz="0 1 0"/>
-        <limit effort="500" velocity="100" lower="${-PI}" upper="${PI}"/>
+        <limit effort="5000" velocity="100" lower="${-PI}" upper="${PI}"/>
         <dynamics damping="${joint_damping}" friction="${joint_friction}"/>
     </joint>
@@ -94,5 +94,5 @@
         <origin xyz="0 0 -${(L_sh)}"/>
         <axis xyz="0 1 0"/>
-        <limit effort="500" velocity="100" lower="${-PI}" upper="${PI}"/>
+        <limit effort="5000" velocity="100" lower="${-PI}" upper="${PI}"/>
         <dynamics damping="${joint_damping}" friction="${joint_friction}"/>
     </joint>

File: src/lookchoop_description/urdf/robot_params.xacro (robot description, xacro)
@@ -23,5 +23,5 @@
     <xacro:property name="mass_thigh" value="0.835"/>
     <xacro:property name="mass_shank" value="0.501"/>
-    <xacro:property name="mass_foot" value="60.159"/>
+    <xacro:property name="mass_foot" value="0.159"/>
     <xacro:property name="mass_toe" value="0.49"/>
     <xacro:property name="joint_damping" value="0.1"/>
